File: chok_boi/docs/chok_boi.sch (EAGLE design)
At the start: 97 parts, among them U1 MPU-6000, U2 DRV8835

Commit message: Improve upper half board placement
Parts:
- removed C_REC_LD, C_REC_LF, C_REC_LH, C_REC_RD, C_REC_RF, C_REC_RH: 0.1uF, SparkFun:CAP0603-CAP
Connections:
- net A3.3V: no longer C_REC_LD.1, C_REC_LF.1, C_REC_LH.1, C_REC_RD.1, C_REC_RF.1, C_REC_RH.1
- net AGND: no longer C_REC_LD.2, C_REC_LF.2, C_REC_LH.2, C_REC_RD.2, C_REC_RF.2, C_REC_RH.2
- net EM_D: now also U$5.PA7; no longer U$5.PA5
- net EM_H: now also U$5.PB0; no longer U$5.PA7
- net REC_RH: now also U$5.PA5; no longer U$5.PB0
Changed lines of the file:
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@@
 <part name="R_RLH" library="SparkFun-Passives" deviceset="RESISTOR" device="0603-RES" value="1.8k"/>
 <part name="U1" library="SparkFun-Sensors" deviceset="MPU-6000" device=""/>
-<part name="C_REC_LD" library="SparkFun" deviceset="CAP" device="0603-CAP" value="0.1uF"/>
-<part name="C_REC_RD" library="SparkFun" deviceset="CAP" device="0603-CAP" value="0.1uF"/>
-<part name="C_REC_RF" library="SparkFun" deviceset="CAP" device="0603-CAP" value="0.1uF"/>
-<part name="C_REC_RH" library="SparkFun" deviceset="CAP" device="0603-CAP" value="0.1uF"/>
-<part name="C_REC_LH" library="SparkFun" deviceset="CAP" device="0603-CAP" value="0.1uF"/>
-<part name="C_REC_LF" library="SparkFun" deviceset="CAP" device="0603-CAP" value="0.1uF"/>
 <part name="C_GY_REG" library="SparkFun" deviceset="CAP" device="0603-CAP" value="0.1uF"/>
 <part name="C_GY_CP" library="SparkFun" deviceset="CAP" device="0603-CAP" value="2.2nF"/>
@@
 <instance part="R_RLH" gate="G$1" x="350.52" y="40.64" rot="R90"/>
 <instance part="U1" gate="G$1" x="60.96" y="-78.74"/>
-<instance part="C_REC_LD" gate="G$1" x="203.2" y="58.42"/>
-<instance part="C_REC_RD" gate="G$1" x="238.76" y="58.42"/>
-<instance part="C_REC_RF" gate="G$1" x="276.86" y="58.42"/>
-<instance part="C_REC_RH" gate="G$1" x="317.5" y="58.42"/>
-<instance part="C_REC_LH" gate="G$1" x="358.14" y="58.42"/>
-<instance part="C_REC_LF" gate="G$1" x="170.18" y="58.42"/>
 <instance part="C_GY_REG" gate="G$1" x="22.86" y="-93.98"/>
 <instance part="C_GY_CP" gate="G$1" x="35.56" y="-93.98"/>
@@
 <pinref part="R_RRD" gate="G$1" pin="1"/>
 <wire x1="231.14" y1="35.56" x2="231.14" y2="25.4" width="0.1524" layer="91"/>
-<wire x1="269.24" y1="25.4" x2="238.76" y2="25.4" width="0.1524" layer="91"/>
+<wire x1="269.24" y1="25.4" x2="231.14" y2="25.4" width="0.1524" layer="91"/>
 <pinref part="R_RLD" gate="G$1" pin="1"/>
-<wire x1="238.76" y1="25.4" x2="231.14" y2="25.4" width="0.1524" layer="91"/>
 <wire x1="195.58" y1="35.56" x2="195.58" y2="25.4" width="0.1524" layer="91"/>
-<wire x1="231.14" y1="25.4" x2="203.2" y2="25.4" width="0.1524" layer="91"/>
+<wire x1="231.14" y1="25.4" x2="195.58" y2="25.4" width="0.1524" layer="91"/>
 <junction x="231.14" y="25.4"/>
 <pinref part="R_RLF" gate="G$1" pin="1"/>
-<wire x1="203.2" y1="25.4" x2="195.58" y2="25.4" width="0.1524" layer="91"/>
 <wire x1="162.56" y1="35.56" x2="162.56" y2="25.4" width="0.1524" layer="91"/>
-<wire x1="195.58" y1="25.4" x2="170.18" y2="25.4" width="0.1524" layer="91"/>
+<wire x1="195.58" y1="25.4" x2="162.56" y2="25.4" width="0.1524" layer="91"/>
 <junction x="195.58" y="25.4"/>
 <pinref part="AGND1" gate="VR1" pin="AGND"/>
 <junction x="162.56" y="25.4"/>
 <pinref part="R_RRH" gate="G$1" pin="1"/>
-<wire x1="170.18" y1="25.4" x2="162.56" y2="25.4" width="0.1524" layer="91"/>
 <wire x1="309.88" y1="35.56" x2="309.88" y2="25.4" width="0.1524" layer="91"/>
-<wire x1="309.88" y1="25.4" x2="276.86" y2="25.4" width="0.1524" layer="91"/>
+<wire x1="309.88" y1="25.4" x2="269.24" y2="25.4" width="0.1524" layer="91"/>
 <junction x="269.24" y="25.4"/>
 <pinref part="R_RLH" gate="G$1" pin="1"/>
-<wire x1="276.86" y1="25.4" x2="269.24" y2="25.4" width="0.1524" layer="91"/>
 <wire x1="350.52" y1="35.56" x2="350.52" y2="25.4" width="0.1524" layer="91"/>
-<wire x1="350.52" y1="25.4" x2="317.5" y2="25.4" width="0.1524" layer="91"/>
+<wire x1="350.52" y1="25.4" x2="309.88" y2="25.4" width="0.1524" layer="91"/>
 <junction x="309.88" y="25.4"/>
-<pinref part="C_REC_LF" gate="G$1" pin="2"/>
-<wire x1="317.5" y1="25.4" x2="309.88" y2="25.4" width="0.1524" layer="91"/>
-<wire x1="170.18" y1="55.88" x2="170.18" y2="25.4" width="0.1524" layer="91"/>
-<junction x="170.18" y="25.4"/>
-<pinref part="C_REC_LD" gate="G$1" pin="2"/>
-<wire x1="203.2" y1="55.88" x2="203.2" y2="25.4" width="0.1524" layer="91"/>
-<junction x="203.2" y="25.4"/>
-<pinref part="C_REC_RD" gate="G$1" pin="2"/>
-<wire x1="238.76" y1="55.88" x2="238.76" y2="25.4" width="0.1524" layer="91"/>
-<junction x="238.76" y="25.4"/>
-<pinref part="C_REC_RF" gate="G$1" pin="2"/>
-<wire x1="276.86" y1="55.88" x2="276.86" y2="25.4" width="0.1524" layer="91"/>
-<junction x="276.86" y="25.4"/>
-<pinref part="C_REC_RH" gate="G$1" pin="2"/>
-<wire x1="317.5" y1="55.88" x2="317.5" y2="25.4" width="0.1524" layer="91"/>
-<junction x="317.5" y="25.4"/>
-<pinref part="C_REC_LH" gate="G$1" pin="2"/>
-<wire x1="358.14" y1="55.88" x2="358.14" y2="25.4" width="0.1524" layer="91"/>
-<wire x1="358.14" y1="25.4" x2="350.52" y2="25.4" width="0.1524" layer="91"/>
-<junction x="350.52" y="25.4"/>
 </segment>
 <segment>
@@
 <wire x1="147.32" y1="71.12" x2="162.56" y2="71.12" width="0.1524" layer="91"/>
 <pinref part="U$9" gate="G$1" pin="C"/>
-<wire x1="162.56" y1="71.12" x2="170.18" y2="71.12" width="0.1524" layer="91"/>
-<wire x1="170.18" y1="71.12" x2="195.58" y2="71.12" width="0.1524" layer="91"/>
-<wire x1="195.58" y1="71.12" x2="203.2" y2="71.12" width="0.1524" layer="91"/>
-<wire x1="203.2" y1="71.12" x2="231.14" y2="71.12" width="0.1524" layer="91"/>
-<wire x1="231.14" y1="71.12" x2="238.76" y2="71.12" width="0.1524" layer="91"/>
-<wire x1="238.76" y1="71.12" x2="269.24" y2="71.12" width="0.1524" layer="91"/>
+<wire x1="162.56" y1="71.12" x2="195.58" y2="71.12" width="0.1524" layer="91"/>
+<wire x1="195.58" y1="71.12" x2="231.14" y2="71.12" width="0.1524" layer="91"/>
+<wire x1="231.14" y1="71.12" x2="269.24" y2="71.12" width="0.1524" layer="91"/>
 <wire x1="269.24" y1="71.12" x2="269.24" y2="63.5" width="0.1524" layer="91"/>
 <pinref part="U$8" gate="G$1" pin="C"/>
@@
 <pinref part="U$20" gate="G$1" pin="C"/>
 <wire x1="309.88" y1="63.5" x2="309.88" y2="71.12" width="0.1524" layer="91"/>
-<wire x1="309.88" y1="71.12" x2="276.86" y2="71.12" width="0.1524" layer="91"/>
+<wire x1="309.88" y1="71.12" x2="269.24" y2="71.12" width="0.1524" layer="91"/>
 <junction x="269.24" y="71.12"/>
 <pinref part="U$21" gate="G$1" pin="C"/>
-<wire x1="276.86" y1="71.12" x2="269.24" y2="71.12" width="0.1524" layer="91"/>
 <wire x1="350.52" y1="63.5" x2="350.52" y2="71.12" width="0.1524" layer="91"/>
-<wire x1="350.52" y1="71.12" x2="317.5" y2="71.12" width="0.1524" layer="91"/>
+<wire x1="350.52" y1="71.12" x2="309.88" y2="71.12" width="0.1524" layer="91"/>
 <junction x="309.88" y="71.12"/>
-<pinref part="C_REC_LF" gate="G$1" pin="1"/>
-<wire x1="317.5" y1="71.12" x2="309.88" y2="71.12" width="0.1524" layer="91"/>
-<wire x1="170.18" y1="63.5" x2="170.18" y2="71.12" width="0.1524" layer="91"/>
-<junction x="170.18" y="71.12"/>
-<pinref part="C_REC_LD" gate="G$1" pin="1"/>
-<wire x1="203.2" y1="63.5" x2="203.2" y2="71.12" width="0.1524" layer="91"/>
-<junction x="203.2" y="71.12"/>
-<pinref part="C_REC_RD" gate="G$1" pin="1"/>
-<wire x1="238.76" y1="63.5" x2="238.76" y2="71.12" width="0.1524" layer="91"/>
-<junction x="238.76" y="71.12"/>
-<pinref part="C_REC_RF" gate="G$1" pin="1"/>
-<wire x1="276.86" y1="63.5" x2="276.86" y2="71.12" width="0.1524" layer="91"/>
-<junction x="276.86" y="71.12"/>
-<pinref part="C_REC_RH" gate="G$1" pin="1"/>
-<wire x1="317.5" y1="63.5" x2="317.5" y2="71.12" width="0.1524" layer="91"/>
-<junction x="317.5" y="71.12"/>
-<pinref part="C_REC_LH" gate="G$1" pin="1"/>
-<wire x1="358.14" y1="63.5" x2="358.14" y2="71.12" width="0.1524" layer="91"/>
-<wire x1="358.14" y1="71.12" x2="350.52" y2="71.12" width="0.1524" layer="91"/>
-<junction x="350.52" y="71.12"/>
 </segment>
 <segment>
@@
 </segment>
 <segment>
-<pinref part="U$5" gate="G$1" pin="PA5"/>
-<wire x1="-101.6" y1="-109.22" x2="-101.6" y2="-114.3" width="0.1524" layer="91"/>
-<label x="-101.6" y="-114.3" size="0.889" layer="95" rot="R270" xref="yes"/>
+<pinref part="U$5" gate="G$1" pin="PA7"/>
+<wire x1="-96.52" y1="-109.22" x2="-96.52" y2="-114.3" width="0.1524" layer="91"/>
+<label x="-96.52" y="-114.3" size="0.8128" layer="95" rot="R270" xref="yes"/>
 </segment>
 </net>
@@
 </segment>
 <segment>
-<pinref part="U$5" gate="G$1" pin="PB0"/>
-<wire x1="-88.9" y1="-109.22" x2="-88.9" y2="-114.3" width="0.1524" layer="91"/>
-<label x="-88.9" y="-114.3" size="0.8128" layer="95" rot="R270" xref="yes"/>
+<pinref part="U$5" gate="G$1" pin="PA5"/>
+<wire x1="-101.6" y1="-109.22" x2="-101.6" y2="-114.3" width="0.1524" layer="91"/>
+<label x="-101.6" y="-114.3" size="0.889" layer="95" rot="R270" xref="yes"/>
 </segment>
 </net>
@@
 </segment>
 <segment>
-<pinref part="U$5" gate="G$1" pin="PA7"/>
-<wire x1="-96.52" y1="-109.22" x2="-96.52" y2="-114.3" width="0.1524" layer="91"/>
-<label x="-96.52" y="-114.3" size="0.8128" layer="95" rot="R270" xref="yes"/>
-</segment>
-</net>
+<pinref part="U$5" gate="G$1" pin="PB0"/>
+<wire x1="-88.9" y1="-109.22" x2="-88.9" y2="-114.3" width="0.1524" layer="91"/>
+<label x="-88.9" y="-114.3" size="0.8128" layer="95" rot="R270" xref="yes"/>
+</segment>
+</net>

Commit message: In middle of reworking traces
Parts:
- R_BOOT1: device SparkFun-Passives:RESISTOR0603-RES -> SparkFun-Passives:RESISTOR0402-RES
Connections:
- net EM_H: now also U$5.PA6; no longer U$5.PB0
- net REC_LD: now also U$5.PC5; no longer U$5.PC4
- net REC_LF: now also U$5.PB1; no longer U$5.PC5
- net REC_LH: now also U$5.PB0; no longer U$5.PB1
- net REC_RD: now also U$5.PC4; no longer U$5.PA6
- net SS1: now also U$5.PC7; no longer U$5.PC8
Changed lines of the file:
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@@
 <part name="SERIAL1" library="pinhead" deviceset="PINHD-1X4" device=""/>
 <part name="SERIAL2" library="pinhead" deviceset="PINHD-1X4" device=""/>
-<part name="R_BOOT1" library="SparkFun-Passives" deviceset="RESISTOR" device="0603-RES" value="47k"/>
+<part name="R_BOOT1" library="SparkFun-Passives" deviceset="RESISTOR" device="0402-RES" value="47k"/>
 <part name="U$18" library="sfh4550 _ teft4300" deviceset="EMITTER" device=""/>
 <part name="U$19" library="sfh4550 _ teft4300" deviceset="EMITTER" device=""/>
@@
 </segment>
 <segment>
-<pinref part="U$5" gate="G$1" pin="PC5"/>
-<wire x1="-91.44" y1="-109.22" x2="-91.44" y2="-114.3" width="0.1524" layer="91"/>
-<label x="-91.44" y="-114.3" size="0.889" layer="95" rot="R270" xref="yes"/>
+<pinref part="U$5" gate="G$1" pin="PB1"/>
+<wire x1="-86.36" y1="-109.22" x2="-86.36" y2="-114.3" width="0.1524" layer="91"/>
+<label x="-86.36" y="-114.3" size="0.8128" layer="95" rot="R270" xref="yes"/>
 </segment>
 </net>
@@
 </segment>
 <segment>
-<pinref part="U$5" gate="G$1" pin="PC4"/>
-<wire x1="-93.98" y1="-109.22" x2="-93.98" y2="-114.3" width="0.1524" layer="91"/>
-<label x="-93.98" y="-114.3" size="0.889" layer="95" rot="R270" xref="yes"/>
+<pinref part="U$5" gate="G$1" pin="PC5"/>
+<wire x1="-91.44" y1="-109.22" x2="-91.44" y2="-114.3" width="0.1524" layer="91"/>
+<label x="-91.44" y="-114.3" size="0.889" layer="95" rot="R270" xref="yes"/>
 </segment>
 </net>
@@
 </segment>
 <segment>
-<pinref part="U$5" gate="G$1" pin="PA6"/>
-<wire x1="-99.06" y1="-109.22" x2="-99.06" y2="-114.3" width="0.1524" layer="91"/>
-<label x="-99.06" y="-114.3" size="0.889" layer="95" rot="R270" xref="yes"/>
+<pinref part="U$5" gate="G$1" pin="PC4"/>
+<wire x1="-93.98" y1="-109.22" x2="-93.98" y2="-114.3" width="0.1524" layer="91"/>
+<label x="-93.98" y="-114.3" size="0.889" layer="95" rot="R270" xref="yes"/>
 </segment>
 </net>
@@
 </segment>
 <segment>
-<pinref part="U$5" gate="G$1" pin="PB1"/>
-<wire x1="-86.36" y1="-109.22" x2="-86.36" y2="-114.3" width="0.1524" layer="91"/>
-<label x="-86.36" y="-114.3" size="0.8128" layer="95" rot="R270" xref="yes"/>
+<pinref part="U$5" gate="G$1" pin="PB0"/>
+<wire x1="-88.9" y1="-109.22" x2="-88.9" y2="-114.3" width="0.1524" layer="91"/>
+<label x="-88.9" y="-114.3" size="0.8128" layer="95" rot="R270" xref="yes"/>
 </segment>
 </net>
@@
 </segment>
 <segment>
-<pinref part="U$5" gate="G$1" pin="PB0"/>
-<wire x1="-88.9" y1="-109.22" x2="-88.9" y2="-114.3" width="0.1524" layer="91"/>
-<label x="-88.9" y="-114.3" size="0.8128" layer="95" rot="R270" xref="yes"/>
+<pinref part="U$5" gate="G$1" pin="PA6"/>
+<wire x1="-99.06" y1="-109.22" x2="-99.06" y2="-114.3" width="0.1524" layer="91"/>
+<label x="-99.06" y="-114.3" size="0.889" layer="95" rot="R270" xref="yes"/>
 </segment>
 </net>
@@
 </segment>
 <segment>
-<pinref part="U$5" gate="G$1" pin="PC8"/>
-<wire x1="-55.88" y1="-76.2" x2="-50.8" y2="-76.2" width="0.1524" layer="91"/>
-<label x="-50.8" y="-76.2" size="0.8128" layer="95" xref="yes"/>
-</segment>
-</net>
+<pinref part="U$5" gate="G$1" pin="PC7"/>
+<wire x1="-55.88" y1="-78.74" x2="-50.8" y2="-78.74" width="0.1524" layer="91"/>
+<label x="-50.8" y="-78.74" size="0.889" layer="95" xref="yes"/>
+</segment>
+</net>

Commit message: More routing
Parts:
- added C1: (no value), SparkFun:CAP1210
- C_5V2, C_BAT2: value 100uF -> 47uF; device SparkFun-Passives:CAP1206 -> SparkFun:CAP1210
- C_MB: device SparkFun:CAP0603-CAP -> Volks73-Kemet:T491X107K025AT
Connections:
- net BATTERY: now also C_MB.A; no longer C_MB.2
- net EM_LF: now also U$5.PA11; no longer U$5.PC6
- net LED1: now also U$5.PC6; no longer U$5.PA11
- net MGND: now also C_MB.C; no longer C_MB.1
- net PWMLB: now also U$5.PB6; no longer U$5.PB7
- net PWMLF: now also U$5.PB7; no longer U$5.PB6
Changed lines of the file:
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@@
 <part name="U$5" library="STM32F10x F4xx" deviceset="STM32F405/415_LQFP64" device=""/>
 <part name="REC_LF" library="sfh4550 _ teft4300" deviceset="RECEIVER" device=""/>
-<part name="C_BAT2" library="SparkFun-Passives" deviceset="CAP" device="1206" value="100uF"/>
+<part name="C_BAT2" library="SparkFun" deviceset="CAP" device="1210" value="47uF"/>
 <part name="R_RLF" library="SparkFun-Passives" deviceset="RESISTOR" device="0603-RES" value="1.8k"/>
 <part name="U$7" library="sfh4550 _ teft4300" deviceset="RECEIVER" device=""/>
@@
 <part name="L1" library="SparkFun-Passives" deviceset="INDUCTOR" device="1007" value="10uH"/>
 <part name="C_BAT1" library="SparkFun-Capacitors" deviceset="CAP" device="0603-CAP" value="0.1uF"/>
-<part name="C_5V2" library="SparkFun-Passives" deviceset="CAP" device="1206" value="100uF"/>
+<part name="C_5V2" library="SparkFun" deviceset="CAP" device="1210" value="47uF"/>
 <part name="C_ELF1" library="SparkFun-Capacitors" deviceset="CAP" device="0603-CAP" value="4.7uF"/>
 <part name="C_ELF2" library="SparkFun-Capacitors" deviceset="CAP" device="0603-CAP" value="0.1uF"/>
@@
 <part name="C_M1" library="SparkFun" deviceset="CAP" device="0603-CAP" value="0.1uF"/>
 <part name="C_M2" library="SparkFun" deviceset="CAP" device="0603-CAP" value="0.1uF"/>
-<part name="C_MB" library="SparkFun" deviceset="CAP" device="0603-CAP" value="100uF"/>
+<part name="C_MB" library="Volks73-Kemet" deviceset="T491?*" device="X" technology="107K025AT" value="100uF"/>
+<part name="C1" library="SparkFun" deviceset="CAP" device="1210"/>
 </parts>
 <sheets>
@@
 <instance part="C_M1" gate="G$1" x="-165.1" y="-177.8" rot="R180"/>
 <instance part="C_M2" gate="G$1" x="-177.8" y="-177.8" rot="R180"/>
-<instance part="C_MB" gate="G$1" x="-187.96" y="-177.8" rot="R180"/>
+<instance part="C_MB" gate="G$1" x="-190.5" y="-180.34"/>
+<instance part="C1" gate="G$1" x="-193.04" y="-149.86"/>
 </instances>
 <busses>
@@
 <label x="-195.58" y="-170.18" size="0.889" layer="95" rot="R180" xref="yes"/>
 <pinref part="C_M2" gate="G$1" pin="2"/>
-<wire x1="-177.8" y1="-170.18" x2="-187.96" y2="-170.18" width="0.1524" layer="91"/>
-<wire x1="-187.96" y1="-170.18" x2="-195.58" y2="-170.18" width="0.1524" layer="91"/>
+<wire x1="-177.8" y1="-170.18" x2="-190.5" y2="-170.18" width="0.1524" layer="91"/>
+<wire x1="-190.5" y1="-170.18" x2="-195.58" y2="-170.18" width="0.1524" layer="91"/>
 <wire x1="-177.8" y1="-175.26" x2="-177.8" y2="-170.18" width="0.1524" layer="91"/>
 <junction x="-177.8" y="-170.18"/>
-<pinref part="C_MB" gate="G$1" pin="2"/>
-<wire x1="-187.96" y1="-175.26" x2="-187.96" y2="-170.18" width="0.1524" layer="91"/>
-<junction x="-187.96" y="-170.18"/>
+<pinref part="C_MB" gate="G$1" pin="A"/>
+<wire x1="-190.5" y1="-175.26" x2="-190.5" y2="-170.18" width="0.1524" layer="91"/>
+<junction x="-190.5" y="-170.18"/>
 </segment>
 </net>
@@
 <net name="PWMLB" class="0">
 <segment>
+<pinref part="U2" gate="G$1" pin="AIN1/PH"/>
+<wire x1="-152.4" y1="-177.8" x2="-154.94" y2="-177.8" width="0.1524" layer="91"/>
+<label x="-154.94" y="-177.8" size="0.889" layer="95" rot="R180" xref="yes"/>
+</segment>
+<segment>
+<pinref part="U$5" gate="G$1" pin="PB6"/>
+<wire x1="-96.52" y1="-35.56" x2="-96.52" y2="-30.48" width="0.1524" layer="91"/>
+<label x="-96.52" y="-30.48" size="0.889" layer="95" rot="R90" xref="yes"/>
+</segment>
+</net>
+<net name="PWMLF" class="0">
+<segment>
+<pinref part="U2" gate="G$1" pin="AIN2/EN"/>
+<wire x1="-152.4" y1="-180.34" x2="-154.94" y2="-180.34" width="0.1524" layer="91"/>
+<label x="-154.94" y="-180.34" size="0.889" layer="95" rot="R180" xref="yes"/>
+</segment>
+<segment>
 <pinref part="U$5" gate="G$1" pin="PB7"/>
 <wire x1="-99.06" y1="-35.56" x2="-99.06" y2="-30.48" width="0.1524" layer="91"/>
 <label x="-99.06" y="-30.48" size="0.889" layer="95" rot="R90" xref="yes"/>
-</segment>
-<segment>
-<pinref part="U2" gate="G$1" pin="AIN1/PH"/>
-<wire x1="-152.4" y1="-177.8" x2="-154.94" y2="-177.8" width="0.1524" layer="91"/>
-<label x="-154.94" y="-177.8" size="0.889" layer="95" rot="R180" xref="yes"/>
-</segment>
-</net>
-<net name="PWMLF" class="0">
-<segment>
-<pinref part="U$5" gate="G$1" pin="PB6"/>
-<wire x1="-96.52" y1="-35.56" x2="-96.52" y2="-30.48" width="0.1524" layer="91"/>
-<label x="-96.52" y="-30.48" size="0.889" layer="95" rot="R90" xref="yes"/>
-</segment>
-<segment>
-<pinref part="U2" gate="G$1" pin="AIN2/EN"/>
-<wire x1="-152.4" y1="-180.34" x2="-154.94" y2="-180.34" width="0.1524" layer="91"/>
-<label x="-154.94" y="-180.34" size="0.889" layer="95" rot="R180" xref="yes"/>
 </segment>
 </net>
@@
 <pinref part="C_M1" gate="G$1" pin="1"/>
 <wire x1="-165.1" y1="-190.5" x2="-177.8" y2="-190.5" width="0.1524" layer="91"/>
-<wire x1="-177.8" y1="-190.5" x2="-187.96" y2="-190.5" width="0.1524" layer="91"/>
-<wire x1="-187.96" y1="-190.5" x2="-198.12" y2="-190.5" width="0.1524" layer="91"/>
+<wire x1="-177.8" y1="-190.5" x2="-190.5" y2="-190.5" width="0.1524" layer="91"/>
+<wire x1="-190.5" y1="-190.5" x2="-198.12" y2="-190.5" width="0.1524" layer="91"/>
 <wire x1="-165.1" y1="-182.88" x2="-165.1" y2="-190.5" width="0.1524" layer="91"/>
 <junction x="-165.1" y="-190.5"/>
@@
 <wire x1="-177.8" y1="-182.88" x2="-177.8" y2="-190.5" width="0.1524" layer="91"/>
 <junction x="-177.8" y="-190.5"/>
-<pinref part="C_MB" gate="G$1" pin="1"/>
-<wire x1="-187.96" y1="-182.88" x2="-187.96" y2="-190.5" width="0.1524" layer="91"/>
-<junction x="-187.96" y="-190.5"/>
+<pinref part="C_MB" gate="G$1" pin="C"/>
+<wire x1="-190.5" y1="-185.42" x2="-190.5" y2="-190.5" width="0.1524" layer="91"/>
+<junction x="-190.5" y="-190.5"/>
 </segment>
 </net>
 <net name="EM_LF" class="0">
-<segment>
-<pinref part="U$5" gate="G$1" pin="PC6"/>
-<wire x1="-55.88" y1="-81.28" x2="-50.8" y2="-81.28" width="0.1524" layer="91"/>
-<label x="-50.8" y="-81.28" size="0.889" layer="95" xref="yes"/>
-</segment>
 <segment>
 <pinref part="R_ELF_PD" gate="G$1" pin="2"/>
@@
 <wire x1="157.48" y1="-66.04" x2="144.78" y2="-66.04" width="0.1524" layer="91"/>
 <junction x="144.78" y="-66.04"/>
+</segment>
+<segment>
+<pinref part="U$5" gate="G$1" pin="PA11"/>
+<wire x1="-55.88" y1="-63.5" x2="-50.8" y2="-63.5" width="0.1524" layer="91"/>
+<label x="-50.8" y="-63.5" size="0.889" layer="95" xref="yes"/>
 </segment>
 </net>
@@
 <net name="LED1" class="0">
 <segment>
-<pinref part="U$5" gate="G$1" pin="PA11"/>
-<wire x1="-55.88" y1="-63.5" x2="-50.8" y2="-63.5" width="0.1524" layer="91"/>
-<label x="-50.8" y="-63.5" size="0.889" layer="95" xref="yes"/>
-</segment>
-<segment>
 <pinref part="LED1" gate="G$1" pin="A"/>
 <wire x1="-180.34" y1="27.94" x2="-180.34" y2="33.02" width="0.1524" layer="91"/>
 <label x="-180.34" y="33.02" size="1.778" layer="95" rot="R90" xref="yes"/>
 </segment>
-</net>
+<segment>
+<pinref part="U$5" gate="G$1" pin="PC6"/>
+<wire x1="-55.88" y1="-81.28" x2="-50.8" y2="-81.28" width="0.1524" layer="91"/>
+<label x="-50.8" y="-81.28" size="0.889" layer="95" xref="yes"/>
+</segment>
+</net>
